File: hardware/piHardware/piHardware.kicad_sch (KiCad schematic)
At the start: 0 parts

Commit message: add:必要なコネクタと基盤の追加(未配線)
Parts:
- added A1: RaspberryPi_Pico, Module:RaspberryPi_Pico_Common_Unspecified, symbol MCU_Module:RaspberryPi_Pico
- added D1, D10, D11, D12, D13, D14, D15, D16, D17, D18, D19, D2, D20, D21, D3, D4, D5, D6, D7, D8, D9: LED, LED_THT:LED_D5.0mm, symbol Device:LED
- added J1: ST7735, Connector_PinHeader_2.54mm:PinHeader_1x08_P2.54mm_Vertical, symbol Connector_Generic:Conn_01x08
- added J2: PCM5102A, Connector_PinHeader_2.54mm:PinHeader_1x10_P2.54mm_Vertical, symbol Connector_Generic:Conn_01x10
- added R1, R10, R11, R12, R13, R14, R15, R16, R17, R18, R19, R2, R20, R21, R3, R4, R5, R6, R7, R8, R9: 1.2k, Resistor_THT:R_Axial_DIN0207_L6.3mm_D2.5mm_P7.62mm_Horizontal, symbol Device:R
- added R22, R23, R24, R25, R26: 4.7k, Resistor_THT:R_Axial_DIN0207_L6.3mm_D2.5mm_P7.62mm_Horizontal, symbol Device:R
- added SW1, SW2, SW3, SW4, SW5: SW_Push, Connector_PinHeader_2.54mm:PinHeader_1x02_P2.54mm_Vertical, symbol Switch:SW_Push
Connections:
- new net: D14.2 (A), R14.1
- new net: D3.2 (A), R3.1
- new net: D15.2 (A), R15.1
- new net: D18.2 (A), R18.1
- new net: D21.2 (A), R21.1
- new net: D11.2 (A), R11.1
- new net: D16.2 (A), R16.1
- new net: D20.2 (A), R20.1
- new net: D17.2 (A), R17.1
- new net: D5.2 (A), R5.1
- new net: D1.2 (A), R1.1
- new net: D12.2 (A), R12.1
- new net: D13.2 (A), R13.1
- new net: D7.2 (A), R7.1
- new net: D19.2 (A), R19.1
- new net: D9.2 (A), R9.1
- new net: D8.2 (A), R8.1
- new net: D2.2 (A), R2.1
- new net: D6.2 (A), R6.1
- new net: D4.2 (A), R4.1
- new net: D10.2 (A), R10.1
- new net +3V3: A1.36 (3V3), J1.1 (Pin_1), J1.8 (Pin_8), J2.1 (Pin_1), J2.9 (Pin_9), SW1.1, SW2.1, SW3.1, SW4.1, SW5.1
- new net GND: A1.13 (GND), A1.18 (GND), A1.23 (GND), A1.28 (GND), A1.3 (GND), A1.38 (GND), A1.8 (GND), J1.7 (Pin_7), J2.10 (Pin_10), J2.2 (Pin_2), J2.6 (Pin_6), J2.7 (Pin_7), J2.8 (Pin_8), R22.2, R23.2, R24.2, R25.2, R26.2
- new net LED1: A1.1 (GPIO0), R1.2, R11.2, R16.2, R21.2, R6.2
- new net LED10: A1.12 (GPIO9), D21.1 (K)
- new net LED2: A1.2 (GPIO1), R12.2, R17.2, R2.2, R7.2
- new net LED3: A1.4 (GPIO2), R13.2, R18.2, R3.2, R8.2
- new net LED4: A1.5 (GPIO3), R14.2, R19.2, R4.2, R9.2
- new net LED5: A1.6 (GPIO4), R10.2, R15.2, R20.2, R5.2
- new net LED6: A1.7 (GPIO5), D1.1 (K), D2.1 (K), D3.1 (K), D4.1 (K), D5.1 (K)
- new net LED7: A1.9 (GPIO6), D10.1 (K), D6.1 (K), D7.1 (K), D8.1 (K), D9.1 (K)
- new net LED8: A1.10 (GPIO7), D11.1 (K), D12.1 (K), D13.1 (K), D14.1 (K), D15.1 (K)
- new net LED9: A1.11 (GPIO8), D16.1 (K), D17.1 (K), D18.1 (K), D19.1 (K), D20.1 (K)
- new net MON.A0: A1.16 (GPIO12), J1.4 (Pin_4)
- new net MON.CS: A1.17 (GPIO13), J1.5 (Pin_5)
- new net MON.RES: A1.20 (GPIO15), J1.6 (Pin_6)
- new net MON.SCK: A1.14 (GPIO10), J1.2 (Pin_2)
- new net MON.SDA: A1.15 (GPIO11), J1.3 (Pin_3)
- new net SPK1: A1.29 (GPIO22), J2.3 (Pin_3)
- new net SPK2: A1.27 (GPIO21), J2.4 (Pin_4)
- new net SPK3: A1.26 (GPIO20), J2.5 (Pin_5)
- new net SW1: A1.21 (GPIO16), R22.1, SW1.2
- new net SW2: A1.22 (GPIO17), R23.1, SW2.2
- new net SW3: A1.24 (GPIO18), R24.1, SW3.2
- new net SW4: A1.25 (GPIO19), R25.1, SW4.2
- new net SW5: A1.31 (GPIO26_ADC0), R26.1, SW5.2
- no-connect marks 0 -> 9
