File: hardware/piHardware/piHardware.kicad_pcb (KiCad board)
At the start: 2 copper layers, 150 x 150 mm, 55 parts, among them J1 ST7735, J2 PCM5102A, SW1 SW_Push, SW2 SW_Push, SW3 SW_Push, SW4 SW_Push, SW5 SW_Push

Commit message: add:必要なコネクタと基盤の追加(未配線)(保存ミスを修正済み)
Parts:
- SW1, SW2, SW3, SW4, SW5: footprint Button_Switch_SMD:Nidec_Copal_CAS-120A -> Connector_PinHeader_2.54mm:PinHeader_1x02_P2.54mm_Vertical
- moved J2 39.0 mm to (111.5, 27.1)
