File: hardware/piHardware/piHardware_routed.kicad_sch (KiCad schematic)
At the start: 55 parts, among them J1 ST7735, J2 PCM5102A, SW1 SW_Push, SW2 SW_Push, SW3 SW_Push, SW4 SW_Push, SW5 SW_Push

Commit message: add:スイッチの種類の変更と電源の追加
Parts:
- removed R22, R23, R24, R25, R26: 4.7k, Resistor_THT:R_Axial_DIN0207_L6.3mm_D2.5mm_P7.62mm_Horizontal, symbol Device:R
- added J3: Battery, Connector_PinHeader_2.54mm:PinHeader_1x02_P2.54mm_Vertical, symbol Connector_Generic:Conn_01x02
- D1, D10, D11, D12, D13, D14, D15, D16, D17, D18, D19, D2, D20, D21, D3, D4, D5, D6, D7, D8, D9: footprint LED_THT:LED_D5.0mm -> Connector_JST:JST_XH_B2B-XH-A_1x02_P2.50mm_Vertical
- SW1, SW2, SW3, SW4, SW5: footprint Connector_PinHeader_2.54mm:PinHeader_1x02_P2.54mm_Vertical -> Connector_JST:JST_XH_B2B-XH-A_1x02_P2.50mm_Vertical
Connections:
- net +3V3: no longer SW1.1, SW2.1, SW3.1, SW4.1, SW5.1
- net GND: now also SW1.2, SW2.2, SW3.2, SW4.2, SW5.2, J3.2 (Pin_2)
- net MON.CS: now also A1.20 (GPIO15), J1.6 (Pin_6); no longer A1.17 (GPIO13), J1.5 (Pin_5)
- net MON.RES: now also A1.17 (GPIO13), J1.5 (Pin_5); no longer A1.20 (GPIO15), J1.6 (Pin_6)
- net SW1: now also SW1.1; no longer SW1.2
- net SW2: now also SW2.1; no longer SW2.2
- net SW3: now also SW3.1; no longer SW3.2
- net SW4: now also SW4.1; no longer SW4.2
- net SW5: now also SW5.1; no longer SW5.2
- net battery: now reaches A1.39 (VSYS)
- net battery: now also J3.1 (Pin_1)
- net SPK1 renamed SPK.DIN
- net SPK2 renamed SPK.LCK
- net SPK3 renamed SPK.BCK
- no-connect marks 9 -> 8
Other:
- moved on the sheet: SW1, SW2, SW3, SW4, SW5

Commit message: feat:フットプリントと電源ボタンの追加
Parts:
- added D22: 1N914, Diode_THT:D_DO-35_SOD27_P7.62mm_Horizontal, symbol Diode:1N914
- added R22: 1.2k, Resistor_THT:R_Axial_DIN0207_L6.3mm_D2.5mm_P7.62mm_Horizontal, symbol Device:R
- added SW6: SW_Push, Connector_JST:JST_XH_B2B-XH-A_1x02_P2.50mm_Vertical, symbol Switch:SW_Push
Connections:
- net SPK.BCK: now also J2.3 (Pin_3); no longer J2.5 (Pin_5)
- net SPK.DIN: now also J2.5 (Pin_5); no longer J2.3 (Pin_3)
- net battery: now also R22.1; no longer J3.1 (Pin_1)
- new net: D22.1 (K), SW6.2
- new net: D22.2 (A), J3.1 (Pin_1)
- new net: R22.2, SW6.1
Other:
- moved on the sheet: J1, J3, SW1, SW2, SW3, SW4, SW5

Commit message: fix:抵抗の削除とスイッチダイオードの変更
Parts:
- removed D22: 1N914, Diode_THT:D_DO-35_SOD27_P7.62mm_Horizontal, symbol Diode:1N914
- removed R22: 1.2k, Resistor_THT:R_Axial_DIN0207_L6.3mm_D2.5mm_P7.62mm_Horizontal, symbol Device:R
- removed SW6: SW_Push, Connector_JST:JST_XH_B2B-XH-A_1x02_P2.50mm_Vertical, symbol Switch:SW_Push
- added D23: 1N5817, Diode_THT:D_DO-41_SOD81_P10.16mm_Horizontal, symbol Diode:1N5817
- added SW6: SW_SPST, Connector_JST:JST_XH_B2B-XH-A_1x02_P2.50mm_Vertical, symbol Switch:SW_SPST
Connections:
- net battery: now also SW6.1 (A)
- net at J3.1 (Pin_1): now also D23.2 (A)
- new net: D23.1 (K), SW6.2 (B)
Changed lines of the file:
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@@
 	(wire
 		(pts
-			(xy 210.82 54.61) (xy 208.28 54.61)
-		)
-		(stroke
-			(width 0)
-			(type default)
-		)
-	)
-	(wire
-		(pts
 			(xy 93.98 49.53) (xy 102.87 49.53)
 		)
@@
 	(wire
 		(pts
-			(xy 200.66 54.61) (xy 196.85 54.61)
+			(xy 196.85 54.61) (xy 210.82 54.61)
 		)
 		(stroke
@@
 	)
 	(symbol
+		(lib_id "Diode:1N5817")
+		(at 229.87 54.61 0)
+		(unit 1)
+		(body_style 1)
+		(exclude_from_sim no)
+		(in_bom yes)
+		(on_board yes)
+		(in_pos_files yes)
+		(dnp no)
+		(fields_autoplaced yes)
+		(property "Reference" "D23"
+			(at 229.5525 48.26 0)
+			(show_name no)
+			(do_not_autoplace no)
+			(effects
+				(font
+					(size 1.27 1.27)
+				)
+			)
+		)
+		(property "Value" "1N5817"
+			(at 229.5525 50.8 0)
+			(show_name no)
+			(do_not_autoplace no)
+			(effects
+				(font
+					(size 1.27 1.27)
+				)
+			)
+		)
+		(property "Footprint" "Diode_THT:D_DO-41_SOD81_P10.16mm_Horizontal"
+			(at 229.87 59.055 0)
+			(hide yes)
+			(show_name no)
+			(do_not_autoplace no)
+			(effects
+				(font
+					(size 1.27 1.27)
+				)
+			)
+		)
+		(property "Datasheet" "http://www.vishay.com/docs/88525/1n5817.pdf"
+			(at 229.87 54.61 0)
+			(hide yes)
+			(show_name no)
+			(do_not_autoplace no)
+			(effects
+				(font
+					(size 1.27 1.27)
+				)
+			)
+		)
+		(property "Description" "20V 1A Schottky Barrier Rectifier Diode, DO-41"
+			(at 229.87 54.61 0)
+			(hide yes)
+			(show_name no)
+			(do_not_autoplace no)
+			(effects
+				(font
+					(size 1.27 1.27)
+				)
+			)
+		)
+		(pin "2"
+		)
+		(pin "1"
+		)
+		(instances
+			(project "piHardware_routed"
+				(path "/c3fc6e3f-150c-4e91-b750-21ca7e978f7f"
+					(reference "D23")
+					(unit 1)
+				)
+			)
+		)
+	)
+	(symbol
 		(lib_id "Device:LED")
 		(at 93.98 85.09 90)
@@
 	)
 	(symbol
-		(lib_id "Diode:1N914")
-		(at 229.87 54.61 0)
+		(lib_id "Device:LED")
+		(at 149.86 106.68 90)
 		(unit 1)
 		(body_style 1)
@@
 		(dnp no)
 		(fields_autoplaced yes)
-		(property "Reference" "D22"
-			(at 229.87 48.26 0)
-			(show_name no)
-			(do_not_autoplace no)
-			(effects
-				(font
-					(size 1.27 1.27)
-				)
-			)
-		)
-		(property "Value" "1N914"
-			(at 229.87 50.8 0)
+		(property "Reference" "D20"
+			(at 153.67 106.9974 90)
 			(show_name no)
 			(do_not_autoplace no)
@@
 					(size 1.27 1.27)
 				)
+				(justify right)
 			)
 		)
-		(property "Footprint" "Diode_THT:D_DO-35_SOD27_P7.62mm_Horizontal"
-			(at 229.87 59.055 0)
-			(hide yes)
+		(property "Value" "LED"
+			(at 153.67 109.5374 90)
 			(show_name no)
 			(do_not_autoplace no)
@@
 					(size 1.27 1.27)
 				)
+				(justify right)
 			)
 		)
-		(property "Datasheet" "http://www.vishay.com/docs/85622/1n914.pdf"
-			(at 229.87 54.61 0)
+		(property "Footprint" "Connector_JST:JST_XH_B2B-XH-A_1x02_P2.50mm_Vertical"
+			(at 149.86 106.68 0)
 			(hide yes)
 			(show_name no)
@@
 			)
 		)
-		(property "Description" "100V 0.3A Small Signal Fast Switching Diode, DO-35"
-			(at 229.87 54.61 0)
+		(property "Datasheet" ""
+			(at 149.86 106.68 0)
 			(hide yes)
 			(show_name no)
@@
 			)
 		)
-		(property "Sim.Device" "D"
-			(at 229.87 54.61 0)
+		(property "Description" "Light emitting diode"
+			(at 149.86 106.68 0)
 			(hide yes)
 			(show_name no)
@@
 		)
 		(property "Sim.Pins" "1=K 2=A"
-			(at 229.87 54.61 0)
+			(at 149.86 106.68 0)
 			(hide yes)
 			(show_name no)
@@
 			(project "piHardware_routed"
 				(path "/c3fc6e3f-150c-4e91-b750-21ca7e978f7f"
-					(reference "D22")
+					(reference "D20")
 					(unit 1)
 				)
@@
 	)
 	(symbol
-		(lib_id "Device:LED")
-		(at 149.86 106.68 90)
+		(lib_id "Switch:SW_SPST")
+		(at 215.9 54.61 0)
 		(unit 1)
 		(body_style 1)
@@
 		(dnp no)
 		(fields_autoplaced yes)
-		(property "Reference" "D20"
-			(at 153.67 106.9974 90)
+		(property "Reference" "SW6"
+			(at 215.9 48.26 0)
 			(show_name no)
 			(do_not_autoplace no)
@@
 					(size 1.27 1.27)
 				)
-				(justify right)
 			)
 		)
-		(property "Value" "LED"
-			(at 153.67 109.5374 90)
+		(property "Value" "SW_SPST"
+			(at 215.9 50.8 0)
 			(show_name no)
 			(do_not_autoplace no)
@@
 					(size 1.27 1.27)
 				)
-				(justify right)
 			)
 		)
 		(property "Footprint" "Connector_JST:JST_XH_B2B-XH-A_1x02_P2.50mm_Vertical"
-			(at 149.86 106.68 0)
+			(at 215.9 54.61 0)
 			(hide yes)
 			(show_name no)
@@
 		)
 		(property "Datasheet" ""
-			(at 149.86 106.68 0)
-			(hide yes)
-			(show_name no)
-			(do_not_autoplace no)
-			(effects
-				(font
-					(size 1.27 1.27)
-				)
-			)
-		)
-		(property "Description" "Light emitting diode"
-			(at 149.86 106.68 0)
+			(at 215.9 54.61 0)
 			(hide yes)
 			(show_name no)
@@
 			)
 		)
-		(property "Sim.Pins" "1=K 2=A"
-			(at 149.86 106.68 0)
+		(property "Description" "Single Pole Single Throw (SPST) switch"
+			(at 215.9 54.61 0)
 			(hide yes)
 			(show_name no)
@@
 			(project "piHardware_routed"
 				(path "/c3fc6e3f-150c-4e91-b750-21ca7e978f7f"
-					(reference "D20")
+					(reference "SW6")
 					(unit 1)
 				)
@@
 	(symbol
 		(lib_id "Switch:SW_Push")
-		(at 215.9 54.61 0)
-		(unit 1)
-		(body_style 1)
-		(exclude_from_sim no)
-		(in_bom yes)
-		(on_board yes)
-		(in_pos_files yes)
-		(dnp no)
-		(fields_autoplaced yes)
-		(property "Reference" "SW6"
-			(at 215.9 46.99 0)
-			(show_name no)
-			(do_not_autoplace no)
-			(effects
-				(font
-					(size 1.27 1.27)
-				)
-			)
-		)
-		(property "Value" "SW_Push"
-			(at 215.9 49.53 0)
-			(show_name no)
-			(do_not_autoplace no)
-			(effects
-				(font
-					(size 1.27 1.27)
-				)
-			)
-		)
-		(property "Footprint" "Connector_JST:JST_XH_B2B-XH-A_1x02_P2.50mm_Vertical"
-			(at 215.9 49.53 0)
-			(hide yes)
-			(show_name no)
-			(do_not_autoplace no)
-			(effects
-				(font
-					(size 1.27 1.27)
-				)
-			)
-		)
-		(property "Datasheet" ""
-			(at 215.9 49.53 0)
-			(hide yes)
-			(show_name no)
-			(do_not_autoplace no)
-			(effects
-				(font
-					(size 1.27 1.27)
-				)
-			)
-		)
-		(property "Description" "Push button switch, generic, two pins"
-			(at 215.9 54.61 0)
-			(hide yes)
-			(show_name no)
-			(do_not_autoplace no)
-			(effects
-				(font
-					(size 1.27 1.27)
-				)
-			)
-		)
-		(pin "2"
-		)
-		(pin "1"
-		)
-		(instances
-			(project "piHardware_routed"
-				(path "/c3fc6e3f-150c-4e91-b750-21ca7e978f7f"
-					(reference "SW6")
-					(unit 1)
-				)
-			)
-		)
-	)
-	(symbol
-		(lib_id "Switch:SW_Push")
 		(at 207.01 85.09 270)
 		(unit 1)
@@
 					(unit 1)
 				)
-			)
-		)
-	)
-	(symbol
-		(lib_id "Device:R")
-		(at 204.47 54.61 90)
-		(unit 1)
-		(body_style 1)
-		(exclude_from_sim no)
-		(in_bom yes)
-		(on_board yes)
-		(in_pos_files yes)
-		(dnp no)
-		(fields_autoplaced yes)
-		(property "Reference" "R22"
-			(at 204.47 48.26 90)
-			(show_name no)
-			(do_not_autoplace no)
-			(effects
-				(font
-					(size 1.27 1.27)
-				)
-			)
-		)
-		(property "Value" "1.2k"
-			(at 204.47 50.8 90)
-			(show_name no)
-			(do_not_autoplace no)
-			(effects
-				(font
-					(size 1.27 1.27)
-				)
-			)
-		)
-		(property "Footprint" "Resistor_THT:R_Axial_DIN0207_L6.3mm_D2.5mm_P7.62mm_Horizontal"
-			(at 204.47 56.388 90)
-			(hide yes)
-			(show_name no)
-			(do_not_autoplace no)
-			(effects
-				(font
-					(size 1.27 1.27)
-				)
-			)
-		)
-		(property "Datasheet" ""
-			(at 204.47 54.61 0)
-			(hide yes)
-			(show_name no)
-			(do_not_autoplace no)
-			(effects
-				(font
-					(size 1.27 1.27)
-				)
-			)
-		)
-		(property "Description" "Resistor"
-			(at 204.47 54.61 0)
-			(hide yes)
-			(show_name no)
-			(do_not_autoplace no)
-			(effects
-				(font
-					(size 1.27 1.27)
-				)
-			)
-		)
-		(pin "2"
-		)
-		(pin "1"
-		)
-		(instances
-			(project "piHardware_routed"
-				(path "/c3fc6e3f-150c-4e91-b750-21ca7e978f7f"
-					(reference "R22")
-					(unit 1)
-				)
