File: hardware/piHardware/piHardware_routed.kicad_pcb (KiCad board)
At the start: 2 copper layers, 99.5 x 99.5 mm, 53 parts, among them J1 ST7735, J2 PCM5102A, J3 Battery, SW1 SW_Push, SW2 SW_Push, SW3 SW_Push, SW4 SW_Push, SW5 SW_Push, SW6 SW_SPST

Commit message: add:pepatikiandhole
Parts:
- added REF**: MountingHole_2.2mm_M2, MountingHole:MountingHole_2.2mm_M2, F.Cu at (163.8, 58.0)
- added REF**: MountingHole_2.2mm_M2, MountingHole:MountingHole_2.2mm_M2, F.Cu at (167.0, 117.0)
- added REF**: MountingHole_2.2mm_M2, MountingHole:MountingHole_2.2mm_M2, F.Cu at (107.8, 58.0)
- added REF**: MountingHole_2.2mm_M2, MountingHole:MountingHole_2.2mm_M2, F.Cu at (73.5, 117.0)
Other:
- board text added: "pi焼き職人 designed by pepatiki"
